File: lzIron_RP2040.kicad_sch (KiCad schematic)
At the start: 231 parts, among them J1 USB_C_Receptacle_USB2.0_16P, U1 XC6206PxxxMR, U2 W25Q128JVS, U3 RP2040, U4 SRV05-4, Y1 ABM8-272-T3

Commit message: V1.1
Parts:
- D1, D10, D11, D12, D13, D14, D15, D16, D17, D18, D19, D2, D20, D21, D22, D23, D24, D25, D26, D27, D28, D29, D3, D30, D31, D32, D33, D34, D35, D36, D37, D38, D39, D4, D40, D41, D42, D43, D44, D45, D46, D47, D48, D49, D5, D50, D51, D52, D53, D54, D55, D56, D57, D58, D59, D6, D60, D61, D62, D63, D64, D65, D66, D67, D68, D69, D7, D70, D71, D72, D73, D74, D75, D76, D77, D78, D79, D8, D80, D81, D82, D83, D84, D85, D86, D87, D88, D89, D9: footprint ScottoKeebs_Components:Diode_SOD-123_noref -> ScottoKeebs_Components:Diode_SOD-123_noref2
