File: lzIron_RP2040.kicad_pcb (KiCad board)
At the start: 2 copper layers, 343.7 x 135.1 mm, 237 parts, among them J1 USB_C_Receptacle_USB2.0_16P, U1 XC6206PxxxMR, U2 W25Q128JVS, U3 RP2040, U4 SRV05-4, Y1 ABM8-272-T3

Commit message: V1.1
Parts:
- D1, D10, D11, D12, D13, D14, D15, D16, D17, D18, D19, D2, D20, D21, D22, D23, D24, D25, D26, D27, D28, D29, D3, D30, D31, D32, D33, D34, D35, D36, D37, D38, D39, D4, D40, D41, D42, D43, D44, D45, D46, D47, D48, D49, D5, D50, D51, D52, D53, D54, D55, D56, D57, D58, D59, D6, D60, D61, D62, D63, D64, D65, D66, D67, D68, D69, D7, D70, D71, D72, D73, D74, D75, D76, D77, D78, D79, D8, D80, D81, D82, D83, D84, D85, D86, D87, D88, D89, D9: footprint ScottoKeebs_Components:Diode_SOD-123_noref -> ScottoKeebs_Components:Diode_SOD-123_noref2

Commit message: V1.2
Routing:
- net +3V3: track 87.5 -> 82.6 mm, vias 5 -> 2
- net +1V1: track 23.2 -> 23.4 mm, vias 0 -> 3
Other:
- outline, holes or cut-outs redrawn

Commit message: V1.3
Parts:
- moved LC1 9.48 mm to (318.2, 119.0), turned to -90 degrees
- moved LC3 9.13 mm to (324.4, 128.1), turned to 180 degrees
- moved LC2 8.15 mm to (325.4, 115.6), turned to 180 degrees
- moved ULED2 7.47 mm to (325.0, 119.0), turned to -90 degrees
- moved ULED1 7.36 mm to (320.9, 119.0), turned to -90 degrees
- moved LC4 6.35 mm to (318.2, 125.2), turned to 90 degrees
- moved ULED3 3.20 mm to (325.0, 124.7), turned to -90 degrees
- moved ULED4 2.94 mm to (320.9, 124.7), turned to 90 degrees
Routing:
- net Net-(ULED4-DOUT): track 56.9 -> 65.0 mm
- net Net-(ULED1-DIN): track 31.6 -> 38.2 mm
- net VBUS: track 609.0 -> 611.5 mm, vias 8 -> 10
- net Net-(ULED3-DOUT): track 5.02 -> 6.11 mm
- net Col17: track 187.0 -> 186.1 mm
- net DP: track 227.9 -> 227.1 mm
- net GND: vias 139 -> 140
